Commit message: v4

File: urdf/macros.xacro (robot description, xacro)
@@ -22,10 +22,10 @@
         <visual>
           <geometry>
-            <mesh filename="$(find my_leo)/models/Rocker.dae"/>
+            <mesh filename="file://$(find my_leo)/models/Rocker.dae"/>
           </geometry>
         </visual>
         <collision>
           <geometry>
-            <mesh filename="$(find my_leo)/models/Rocker_outline.stl"/>
+            <mesh filename="file://$(find my_leo)/models/Rocker_outline.stl"/>
           </geometry>
         </collision>
@@ -44,5 +44,5 @@
         <visual>
           <geometry>
-            <mesh filename="$(find my_leo)/models/Wheel${model}.dae"/>
+            <mesh filename="file://$(find my_leo)/models/Wheel${model}.dae"/>
           </geometry>
         </visual>
@@ -61,5 +61,5 @@
         <collision>
           <geometry>
-            <mesh filename="$(find my_leo)/models/Wheel_outline.stl"/>
+            <mesh filename="file://$(find my_leo)/models/Wheel_outline.stl"/>
           </geometry>
         </collision>
@@ -78,5 +78,5 @@
         <visual>
           <geometry>
-            <mesh filename="$(find my_leo)/models/WheelMecanum${model}.dae"/>
+            <mesh filename="file://$(find my_leo)/models/WheelMecanum${model}.dae"/>
           </geometry>
         </visual>
@@ -89,5 +89,5 @@
         <collision>
           <geometry>
-            <mesh filename="$(find my_leo)/models/Mecanum_wheel_outline.stl"/>
+            <mesh filename="file://$(find my_leo)/models/Mecanum_wheel_outline.stl"/>
           </geometry>
         </collision>
@@ -110,10 +110,10 @@
       <visual>
         <geometry>
-          <mesh filename="$(find my_leo)/models/Chassis.dae"/>
+          <mesh filename="file://$(find my_leo)/models/Chassis.dae"/>
         </geometry>
       </visual>
       <collision>
         <geometry>
-          <mesh filename="$(find my_leo)/models/Chassis_outline.stl"/>
+          <mesh filename="file://$(find my_leo)/models/Chassis_outline.stl"/>
         </geometry>
       </collision>
@@ -145,5 +145,5 @@
         <visual>
           <geometry>
-            <mesh filename="$(find my_leo)/models/Antenna.dae"/>
+            <mesh filename="file://$(find my_leo)/models/Antenna.dae"/>
           </geometry>
         </visual>
